Commit message: Small fix in pexod with springs

File: hexapod_models/URDF/pexod_springs.urdf (robot description, URDF)
Before this commit: robot pexod, 19 links, 18 joints
Links:
- link leg_0_3: geometry collision cylinder length=0.115 radius=0.025; collision sphere radius=0.025
- link leg_1_3: geometry collision cylinder length=0.115 radius=0.025; collision sphere radius=0.025
- link leg_2_3: geometry collision cylinder length=0.115 radius=0.025; collision sphere radius=0.025
- link leg_3_3: geometry collision cylinder length=0.115 radius=0.025; collision sphere radius=0.025
- link leg_4_3: geometry collision cylinder length=0.115 radius=0.025; collision sphere radius=0.025
- link leg_5_3: geometry collision cylinder length=0.115 radius=0.025; collision sphere radius=0.025
