Commit message: Updated Pexod URDF model

File: hexapod_models/URDF/pexod.urdf (robot description, URDF)
Before this commit: robot pexod, 19 links, 18 joints
Links:
- removed link body
- added link base_link, mass 1.031; collision box size=0.24 0.2 0.04; visual box size=0.24 0.2 0.04
- link leg_0_3: geometry collision cylinder length=0.115 radius=0.025; collision sphere radius=0.025
- link leg_1_3: geometry collision cylinder length=0.115 radius=0.025; collision sphere radius=0.025
- link leg_2_3: geometry collision cylinder length=0.115 radius=0.025; collision sphere radius=0.025
- link leg_3_3: geometry collision cylinder length=0.115 radius=0.025; collision sphere radius=0.025
- link leg_4_3: geometry collision cylinder length=0.115 radius=0.025; collision sphere radius=0.025
- link leg_5_3: geometry collision cylinder length=0.115 radius=0.025; collision sphere radius=0.025
Joints:
- joint body_leg_0: axis 0 0 -1 -> 0 0 1; parent body -> base_link
- joint body_leg_1: axis 0 0 -1 -> 0 0 1; parent body -> base_link
- joint body_leg_2: axis 0 0 -1 -> 0 0 1; parent body -> base_link
- joint body_leg_3: axis 0 0 -1 -> 0 0 1; parent body -> base_link
- joint body_leg_4: axis 0 0 -1 -> 0 0 1; parent body -> base_link
- joint body_leg_5: axis 0 0 -1 -> 0 0 1; parent body -> base_link
- joint leg_0_1_2: axis -1 0 0 -> 1 0 0
- joint leg_1_1_2: axis -1 0 0 -> 1 0 0
- joint leg_2_1_2: axis -1 0 0 -> 1 0 0
- joint leg_3_1_2: axis 1 0 0 -> -1 0 0
- joint leg_4_1_2: axis 1 0 0 -> -1 0 0
- joint leg_5_1_2: axis 1 0 0 -> -1 0 0

Commit message: New URDF for pexod

File: hexapod_models/URDF/pexod.urdf (robot description, URDF)
Before this commit: robot pexod, 19 links, 18 joints
Links:
- link leg_0_1: geometry collision box size=0.02 0.02 0.06; visual cylinder length=0.06 radius=0.02
- link leg_0_2: geometry collision box size=0.02 0.02 0.085; visual cylinder length=0.085 radius=0.02
- link leg_0_3: mass 0.184 -> 0.04; geometry collision box size=0.025 0.025 0.14; collision sphere radius=0.025
- link leg_1_1: geometry collision box size=0.02 0.02 0.06; visual cylinder length=0.06 radius=0.02
- link leg_1_2: geometry collision box size=0.02 0.02 0.085; visual cylinder length=0.085 radius=0.02
- link leg_1_3: mass 0.184 -> 0.04; geometry collision box size=0.025 0.025 0.14; collision sphere radius=0.025
- link leg_2_1: geometry collision box size=0.02 0.02 0.06; visual cylinder length=0.06 radius=0.02
- link leg_2_2: geometry collision box size=0.02 0.02 0.085; visual cylinder length=0.085 radius=0.02
- link leg_2_3: mass 0.184 -> 0.04; geometry collision box size=0.025 0.025 0.14; collision sphere radius=0.025
- link leg_3_1: geometry collision box size=0.02 0.02 0.06; visual cylinder length=0.06 radius=0.02
- link leg_3_2: geometry collision box size=0.02 0.02 0.085; visual cylinder length=0.085 radius=0.02
- link leg_3_3: mass 0.184 -> 0.04; geometry collision box size=0.025 0.025 0.14; collision sphere radius=0.025
- link leg_4_1: geometry collision box size=0.02 0.02 0.06; visual cylinder length=0.06 radius=0.02
- link leg_4_2: geometry collision box size=0.02 0.02 0.085; visual cylinder length=0.085 radius=0.02
- link leg_4_3: mass 0.184 -> 0.04; geometry collision box size=0.025 0.025 0.14; collision sphere radius=0.025
- link leg_5_1: geometry collision box size=0.02 0.02 0.06; visual cylinder length=0.06 radius=0.02
- link leg_5_2: geometry collision box size=0.02 0.02 0.085; visual cylinder length=0.085 radius=0.02
- link leg_5_3: mass 0.184 -> 0.04; geometry collision box size=0.025 0.025 0.14; collision sphere radius=0.025
Joints:
- joint body_leg_0: origin xyz=-0.14 0.08 0 rpy=0 0 0.3 -> xyz=-0.13 0.04 0 rpy=0 0 0.3
- joint body_leg_2: origin xyz=0.12 0.08 0 rpy=0 0 -0.3 -> xyz=0.11 0.04 0 rpy=0 0 -0.3
- joint body_leg_3: origin xyz=0.12 -0.08 0 rpy=0 0 0.3 -> xyz=0.11 -0.04 0 rpy=0 0 0.3
- joint body_leg_5: origin xyz=-0.14 -0.08 0 rpy=0 0 -0.3 -> xyz=-0.13 -0.04 0 rpy=0 0 -0.3
